Commit message: added neck joint + update control script

File: B.Virtual_Env/robot/urdf/robotis_mini.urdf (robot description, URDF)
Before this commit: robot robotis_mini, 104 links, 103 joints
Joints:
- joint neck_joint: limit (none) -> lower=-1.5707963267948966 upper=1.5707963267948966 effort=0.1 velocity=11.938052083641214; type fixed -> revolute
